Commit message: Fixed issue with mesh loading

File: hcr_description/urdf/hcr.urdf.xacro (robot description, xacro)
@@ -538,3 +538,67 @@
     </plugin>
   </gazebo>
+<gazebo reference="base_link">
+  <material>Gazebo/Orange</material>
+</gazebo>
+<link name="lidar">
+    <inertial>
+            <mass value="0.005" />
+            <inertia ixx="0.01" ixy="0.0" ixz="0"
+            iyy="0.01" iyz="0" izz="0.01" />
+    </inertial>
+    <visual>
+      <geometry>
+        <cylinder radius="0.025" length="0.025"/>
+      </geometry>
+      <material name="white">
+        <color rgba="1 1 1 1"/>
+      </material>
+    </visual>
+    <collision>
+      <geometry>
+          <box size="0.025 0.025 0.025"/>
+      </geometry>
+    </collision>
+  </link>
+  <joint name="lidar_joint" type="fixed">
+    <origin xyz="0.09 0 0.09" rpy="0 0 0"/>
+    <parent link="base_link"/>
+    <child link="lidar"/>
+    <axis xyz="0.0 0.0 1.0"/>
+  </joint>
+<gazebo reference="lidar">
+    <sensor type="gpu_ray" name="head_hokuyo_sensor">
+      <pose>0 0 0 0 0 0</pose>
+      <visualize>true</visualize>
+      <update_rate>40</update_rate>
+      <ray>
+        <scan>
+          <horizontal>
+            <samples>720</samples>
+            <resolution>1</resolution>
+            <min_angle>-1.570796</min_angle>
+            <max_angle>1.570796</max_angle>
+          </horizontal>
+        </scan>
+        <range>
+          <min>0.10</min>
+          <max>10.0</max>
+          <resolution>0.01</resolution>
+        </range>
+        <noise>
+          <type>gaussian</type>
+          <!-- Noise parameters based on published spec for Hokuyo laser
+               achieving "+-30mm" accuracy at range < 10m.  A mean of 0.0m and
+               stddev of 0.01m will put 99.7% of samples within 0.03m of the true
+               reading. -->
+          <mean>0.0</mean>
+          <stddev>0.01</stddev>
+        </noise>
+      </ray>
+      <plugin name="gazebo_ros_head_hokuyo_controller" filename="libgazebo_ros_ray_sensor.so">
+        <topicName>/hcr/laser/scan</topicName>
+        <frameName>lidar</frameName>
+      </plugin>
+    </sensor>
+  </gazebo>
 </robot>

Commit message: Gazebo material

File: hcr_description/urdf/hcr.urdf.xacro (robot description, xacro)
@@ -540,4 +540,19 @@
 <gazebo reference="base_link">
   <material>Gazebo/Orange</material>
+</gazebo>
+<gazebo reference="LinkLeft">
+  <material>Gazebo/Black</material>
+</gazebo>
+<gazebo reference="LinkRight">
+  <material>Gazebo/Black</material>
+</gazebo>
+<gazebo reference="TopBase">
+  <material>Gazebo/Gray</material>
+</gazebo>
+<gazebo reference="Roller">
+  <material>Gazebo/Black</material>
+</gazebo>
+<gazebo reference="UV">
+  <material>Gazebo/Blue</material>
 </gazebo>
 <link name="lidar">

Commit message: Frame view

File: hcr_description/urdf/hcr.urdf.xacro (robot description, xacro)
@@ -4,4 +4,5 @@
      For more information, please see http://wiki.ros.org/sw_urdf_exporter -->
 <robot name="hcr">
+  <link name="base_footprint"/>
   <link
     name="base_link">
@@ -44,4 +45,9 @@
     </collision>
   </link>
+  <joint name="base_joint" type="fixed">
+    <parent link="base_footprint"/>
+    <child link="base_link"/>
+    <origin rpy="0 0 0" xyz="0 0 0.135"/>
+  </joint>
   <link
     name="LinkLeft">

Commit message: Added imu

File: hcr_description/urdf/hcr.urdf.xacro (robot description, xacro)
@@ -589,5 +589,5 @@
   </joint>
 <gazebo reference="lidar">
-    <sensor type="gpu_ray" name="head_hokuyo_sensor">
+    <sensor type="gpu_ray" name="head_lidar_sensor">
       <pose>0 0 0 0 0 0</pose>
       <visualize>true</visualize>
@@ -617,5 +617,5 @@
         </noise>
       </ray>
-      <plugin name="gazebo_ros_head_hokuyo_controller" filename="libgazebo_ros_ray_sensor.so">
+      <plugin name="gazebo_ros_lidar_controller" filename="libgazebo_ros_ray_sensor.so">
         <topicName>/hcr/laser/scan</topicName>
         <frameName>lidar</frameName>
@@ -623,3 +623,93 @@
     </sensor>
   </gazebo>
+  <link name="imu_link">
+  <inertial>
+            <mass value="0.005" />
+            <inertia ixx="0.01" ixy="0.0" ixz="0"
+            iyy="0.01" iyz="0" izz="0.01" />
+    </inertial>
+  <visual>
+    <geometry>
+      <box size="0.01 0.01 0.01"/>
+    </geometry>
+  </visual>
+  <collision>
+    <geometry>
+      <box size="0.01 0.01 0.01"/>
+    </geometry>
+  </collision>
+</link>
+<joint name="imu_joint" type="fixed">
+  <parent link="base_link"/>
+  <child link="imu_link"/>
+  <origin xyz="0 0 0.01"/>
+</joint>
+ <gazebo reference="imu_link">
+  <sensor name="imu_sensor" type="imu">
+   <plugin filename="libgazebo_ros_imu_sensor.so" name="imu_plugin">
+      <ros>
+        <!--namespace>/hcr</namespace-->
+        <remapping>~/out:=imu</remapping>
+      </ros>
+      <initial_orientation_as_reference>false</initial_orientation_as_reference>
+    </plugin>
+    <always_on>true</always_on>
+    <update_rate>100</update_rate>
+    <visualize>true</visualize>
+    <imu>
+      <angular_velocity>
+        <x>
+          <noise type="gaussian">
+            <mean>0.0</mean>
+            <stddev>2e-4</stddev>
+            <bias_mean>0.0000075</bias_mean>
+            <bias_stddev>0.0000008</bias_stddev>
+          </noise>
+        </x>
+        <y>
+          <noise type="gaussian">
+            <mean>0.0</mean>
+            <stddev>2e-4</stddev>
+            <bias_mean>0.0000075</bias_mean>
+            <bias_stddev>0.0000008</bias_stddev>
+          </noise>
+        </y>
+        <z>
+          <noise type="gaussian">
+            <mean>0.0</mean>
+            <stddev>2e-4</stddev>
+            <bias_mean>0.0000075</bias_mean>
+            <bias_stddev>0.0000008</bias_stddev>
+          </noise>
+        </z>
+      </angular_velocity>
+      <linear_acceleration>
+        <x>
+          <noise type="gaussian">
+            <mean>0.0</mean>
+            <stddev>1.7e-2</stddev>
+            <bias_mean>0.1</bias_mean>
+            <bias_stddev>0.001</bias_stddev>
+          </noise>
+        </x>
+        <y>
+          <noise type="gaussian">
+            <mean>0.0</mean>
+            <stddev>1.7e-2</stddev>
+            <bias_mean>0.1</bias_mean>
+            <bias_stddev>0.001</bias_stddev>
+          </noise>
+        </y>
+        <z>
+          <noise type="gaussian">
+            <mean>0.0</mean>
+            <stddev>1.7e-2</stddev>
+            <bias_mean>0.1</bias_mean>
+            <bias_stddev>0.001</bias_stddev>
+          </noise>
+        </z>
+      </linear_acceleration>
+    </imu>
+  </sensor>
+</gazebo>
 </robot>

Commit message: Added localization

File: hcr_description/urdf/hcr.urdf.xacro (robot description, xacro)
@@ -9,5 +9,5 @@
     <inertial>
       <origin
-        xyz="-0.024595 0.00063611 0.010099"
+        xyz="-0.024595 0.00063611 0.038099"
         rpy="0 0 0" />
       <mass
@@ -48,5 +48,5 @@
     <parent link="base_footprint"/>
     <child link="base_link"/>
-    <origin rpy="0 0 0" xyz="0 0 0.135"/>
+    <origin rpy="0 0 0" xyz="0 0 0"/>
   </joint>
   <link
@@ -533,10 +533,10 @@
       <publish_odom>true</publish_odom>
       <publish_odom_tf>true</publish_odom_tf>
-      <!-- <publish_wheel_tf>false</publish_wheel_tf> -->
-      <update_rate>15.0</update_rate>
+      <publish_wheel_tf>true</publish_wheel_tf>
+      <update_rate>30.0</update_rate>
       <left_joint>leftjoint</left_joint>
       <right_joint>rightjoint</right_joint>
-      <wheel_separation>0.5</wheel_separation>
-      <wheel_diameter>0.3</wheel_diameter>
+      <wheel_separation>0.26</wheel_separation>
+      <wheel_diameter>0.078</wheel_diameter>
       <max_wheel_acceleration>0.7</max_wheel_acceleration>
       <max_wheel_torque>8</max_wheel_torque>
